File: STM32_BASED_BOARD.kicad_sch (KiCad schematic)
At the start: 20 parts, among them J1 USB_B_Micro, J2 Conn_01x04_Pin, SW1 SW_SPDT, U1 STM32F103C8T6, U2 AMS1117, Y1 16MHz

Commit message: V1.1
Parts:
- added C12, C13: 20u, Capacitor_SMD:C_0805_2012Metric, symbol Device:C
- added D1: LED, LED_SMD:LED_0603_1608Metric, symbol Device:LED
- added J3, J4: Conn_01x04_Pin, Connector_PinHeader_2.54mm:PinHeader_1x04_P2.54mm_Vertical, symbol Connector:Conn_01x04_Pin
- added R3, R4, R5: 1K5, Resistor_SMD:R_0402_1005Metric, symbol Device:R
- C1, C2, C3, C4: footprint (none) -> Capacitor_SMD:C_0402_1005Metric
- C10, C11, C7, C8, C9: footprint (none) -> Capacitor_SMD:C_0402_1005Metric_Pad0.74x0.62mm_HandSolder
- C5, C6: footprint (none) -> Capacitor_SMD:C_0603_1608Metric
- FB1: footprint (none) -> Inductor_SMD:L_0603_1608Metric
- J1: footprint (none) -> Connector_USB:USB_Micro-B_Wuerth_629105150521
- J2: footprint (none) -> Connector_PinHeader_2.54mm:PinHeader_1x04_P2.54mm_Vertical
- R1, R2: footprint (none) -> Resistor_SMD:R_0402_1005Metric
- SW1: footprint (none) -> Button_Switch_THT:SW_E-Switch_EG2219_DPDT_Angled
- Y1: footprint (none) -> Crystal:Crystal_SMD_3225-4Pin_3.2x2.5mm
Connections:
- net +3.3V: now also U2.2 (VO), C13.1, D1.2 (A), J3.1 (Pin_1), J4.1 (Pin_1), R4.2, R5.2
- net GND: now also U2.1 (ADJ), C12.2, C13.2, J3.4 (Pin_4), J4.4 (Pin_4), R3.2
- net VBUS: now also U2.3 (VI), C12.1
- net I2C_SCL: now reaches U1.21 (PB10)
- net I2C_SCL: now also J4.2 (Pin_2), R4.1
- net I2C_SDA: now reaches U1.22 (PB11)
- net I2C_SDA: now also J4.3 (Pin_3), R5.1
- net USART1_TX: now reaches U1.43 (PB7)
- net USART1_TX: now also J3.2 (Pin_2)
- net USART1_RX: now reaches U1.45 (PB8)
- net USART1_RX: now also J3.3 (Pin_3)
- new net Power_LED_Cathode: D1.1 (K), R3.1
- no-connect marks 2 -> 29
Other:
- note added: "MICROCONTROLLER CIRCUIT"
- note added: "POWER SUPPLY"
- note added: "STM32_BASED_DevBOARD"
- note added: "USB SECTION"
- title: (none) -> Mostafa Bakir
- moved on the sheet: C1, C10, C11, C2, C3, C4, C5, C6, C7, C8, C9, FB1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
